Commit message: ch33: widen the limits of the gripper's mimic joints so they follow the knuckle and MoveIt accepts the start state
gz_ros2_control set the mimic joints from outside; with limits of +-1.57 some sat at the limit instead of +-0.5
and CheckStartStateBounds aborted the approach on rounding noise (flaky). With +-6.3 they read +-0.5 exactly.

Co-Authored-By: Claude Sonnet 5.5 <noreply@anthropic.com>

File: ros2/xtdrone_robotic_arm/urdf/iris_arm.urdf.xacro (robot description, xacro)
@@ -45,5 +45,7 @@
     <xacro:position_joint name="wrist_2_joint"/>
     <xacro:position_joint name="left_knuckle_joint" initial="0.5"/>
-    <!-- the other gripper joints follow left_knuckle_joint (<mimic> in le_arm_gripper.urdf.xacro) -->
+    <!-- the other gripper joints follow left_knuckle_joint (<mimic> in le_arm_gripper.urdf.xacro). Their limits are
+         +-6.3 there, not +-1.57: gz_ros2_control sets them from outside, they sat at the limit (-1.57) instead of
+         +-0.5, and MoveIt then refused the start state ("outside bounds") on rounding noise. -->
     <xacro:macro name="mimic_joint" params="name">
       <joint name="${name}">

File: ros2/xtdrone_robotic_arm/urdf/le_arm_gripper.urdf.xacro (robot description, xacro)
@@ -161,6 +161,6 @@
             xyz="0 0 -1" />
             <limit
-            lower="-1.57"
-            upper="1.57"
+            lower="-6.3"
+            upper="6.3"
             effort="1000"
             velocity="2.0" />
@@ -220,6 +220,6 @@
             xyz="0 0 1" />
             <limit
-            lower="-1.57"
-            upper="1.57"
+            lower="-6.3"
+            upper="6.3"
             effort="1000"
             velocity="2.0" />
@@ -279,6 +279,6 @@
             xyz="0 0 1" />
             <limit
-            lower="-1.57"
-            upper="1.57"
+            lower="-6.3"
+            upper="6.3"
             effort="1000"
             velocity="2.0" />
@@ -338,6 +338,6 @@
             xyz="0 0 1" />
             <limit
-            lower="-1.57"
-            upper="1.57"
+            lower="-6.3"
+            upper="6.3"
             effort="1000"
             velocity="2.0" />
@@ -397,6 +397,6 @@
             xyz="0 0 -1" />
             <limit
-            lower="-1.57"
-            upper="1.57"
+            lower="-6.3"
+            upper="6.3"
             effort="1000"
             velocity="2.0" />
