Commit message: ch32 and ch33 on ArduPilot: iris_arm on the ArduPilot iris with a legs-and-plate collision variant, camera moved back, takeoff and lift checks for ArduPilot; MAVROS system id 255 for RC overrides

File: ros2/xtdrone_robotic_arm/urdf/iris_arm.urdf.xacro (robot description, xacro)
@@ -13,5 +13,5 @@
        ahead, at the object on the table and the gripper) -->
   <joint name="camera_joint" type="fixed">
-    <origin xyz="0.05 0 -0.07" rpy="0 0 0"/>
+    <origin xyz="-0.15 0 -0.07" rpy="0 0 0"/>
     <parent link="base_link"/>
     <child link="camera_link"/>
